File: eth_phy.kicad_sch (KiCad schematic)
At the start: 2 parts, among them J2 RJ45_RB1-125B8G1A, U2 KSZ9031RNXCA

Commit message: develop: Did some stuff. Not sure what I am doing :).
Parts:
- removed J2: RJ45_RB1-125B8G1A, Connector_RJ:RJ45_UDE_RB1-125B8G1A, symbol Connector:RJ45_RB1-125B8G1A
Changed lines of the file:
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@@
-	)
-	(symbol
-		(lib_id "Connector:RJ45_RB1-125B8G1A")
-		(at 53.34 96.52 0)
-		(mirror x)
-		(unit 1)
-		(exclude_from_sim no)
-		(in_bom yes)
-		(on_board yes)
-		(dnp no)
-		(property "Reference" "J2"
-			(at 44.45 99.0601 0)
-			(effects
-				(font
-					(size 1.27 1.27)
-				)
-				(justify right)
-			)
-		)
-		(property "Value" "RJ45_RB1-125B8G1A"
-			(at 44.45 96.5201 0)
-			(effects
-				(font
-					(size 1.27 1.27)
-				)
-				(justify right)
-			)
-		)
-		(property "Footprint" "Connector_RJ:RJ45_UDE_RB1-125B8G1A"
-			(at 54.61 99.06 0)
-			(effects
-				(font
-					(size 1.27 1.27)
-				)
-				(hide yes)
-			)
-		)
-		(property "Datasheet" "https://datasheet.lcsc.com/szlcsc/1901091107_UDE-Corp-RB1-125B8G1A_C363353.pdf"
-			(at 47.244 97.663 0)
-			(effects
-				(font
-					(size 1.27 1.27)
-				)
-				(justify left top)
-				(hide yes)
-			)
-		)
-		(property "Description" "LAN Transformer Jack, RJ45, 10/100/1000 BaseT"
-			(at 53.34 96.52 0)
-			(effects
-				(font
-					(size 1.27 1.27)
-				)
-				(hide yes)
-			)
-		)
-		(pin "R6"
-		)
-		(pin "R7"
-		)
-		(pin "L1"
-		)
-		(pin "SH"
-		)
-		(pin "R3"
-		)
-		(pin "R10"
-		)
-		(pin "R9"
-		)
-		(pin "R8"
-		)
-		(pin "R5"
-		)
-		(pin "L2"
-		)
-		(pin "R4"
-		)
-		(pin "R1"
-		)
-		(pin "L3"
-		)
-		(pin "R2"
-		)
-		(pin "L4"
-		)
-		(instances
-			(project ""
-				(path "/ba4aeeea-982a-4252-9638-c2cfeb24b844/4e28fc7d-4fd5-4314-9908-3f9331eae463"
-					(reference "J2")
-					(unit 1)
-				)
-			)
-		)
 	)
 	(symbol
